Commit message: Add soft-body envs: Pinch-v0 and Write-v0
* add Pinch and Write envs

* pad goal points with 0 to ensure shape

* add error message for missing assets

* remove used imports

* move panda config location to variants

* cleanups, add precompile

* make pinch fingers collide

* fix write bugs, filter for h5 files in level dir

* improve pinch stability

* update pinch asset checksum

* fix panda stick urdf

* update write obs type

* target points xyz->xyzw

* Add panda_stick.srdf

* Simplify searching level files

Co-authored-by: Fanbo Xiang <xiangfanbo@gmail.com>
Co-authored-by: Xinyue Wei <13659185706@163.com>

File: mani_skill2/assets/descriptions/panda_stick.urdf (robot description, URDF)
Before this commit: robot panda, 10 links, 9 joints
Links:
- added link panda_hand_tcp
- link panda_hand: geometry collision capsule length=0.1 radius=0.008; collision mesh filename=franka_description/meshes/collision/hand.stl
Joints:
- added joint panda_hand_tcp_joint: type fixed, parent panda_hand, child panda_hand_tcp, origin xyz=0 0 0.15 rpy=0 0 0
